Commit message: fixing scripts

File: my_robot/urdf/my_robot.xacro (robot description, xacro)
@@ -11,5 +11,5 @@
     <pose>0 0 0.1 0 0 0</pose>
     <inertial>
-      <mass value="1.0"/>
+      <mass value="10.0"/>
       <origin xyz="0.0 0 0" rpy=" 0 0 0"/>
       <inertia
@@ -58,5 +58,5 @@
   <link name='right_wheel'>
     <inertial>
-      <mass value="1.0"/>
+      <mass value="5.0"/>
       <origin xyz="0 0 0" rpy=" 0 1.5707 1.5707"/>
       <inertia
@@ -81,5 +81,5 @@
   <link name='left_wheel'>
     <inertial>
-      <mass value="1.0"/>
+      <mass value="5.0"/>
       <origin xyz="0 0 0" rpy=" 0 1.5707 1.5707"/>
       <inertia
